File: JouleThief/JouleThief.kicad_sch (KiCad schematic)
At the start: 8 parts, among them J1 Screw_Terminal_01x02, J2 Screw_Terminal_01x02, Q1 BC547, Q2 BC547

Commit message: Finished PCB
Parts:
- added D1: LED, LED_THT:LED_D5.0mm_Clear, symbol Device:LED
- added R3: 300, Resistor_THT:R_Axial_DIN0204_L3.6mm_D1.6mm_P7.62mm_Horizontal, symbol Device:R
- added S1: SWITCH-SPDT-PTH-11.6X4.0MM-KIT, SnapEDA Library:SW_1825159-1, symbol SparkFun-Switches:SWITCH-SPDT-PTH-11.6X4.0MM-KIT
Connections:
- net GND: now also R3.2
- net at C1.1, L1.1, Q1.1 (C)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: now also S1.2 (P); no longer J1.2 (Pin_2)
- new net: D1.2 (A), S1.1 (O)
- new net: J1.2 (Pin_2), S1.3 (S)
- new net: D1.1 (K), R3.1
Other:
- moved on the sheet: J1
Changed lines of the file:
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@@
   (junction (at 139.7 110.49) (diameter 0) (color 0 0 0 0)
   )
+  (junction (at 113.03 110.49) (diameter 0) (color 0 0 0 0)
+  )
   (junction (at 139.7 92.71) (diameter 0) (color 0 0 0 0)
   )
@@
   (junction (at 125.73 110.49) (diameter 0) (color 0 0 0 0)
   )
+  (wire (pts (xy 104.775 110.49) (xy 113.03 110.49))
+    (stroke (width 0) (type default) (color 0 0 0 0))
+  )
   (wire (pts (xy 125.73 109.22) (xy 125.73 110.49))
     (stroke (width 0) (type default) (color 0 0 0 0))
@@
     (stroke (width 0) (type default) (color 0 0 0 0))
   )
-  (wire (pts (xy 125.73 110.49) (xy 116.205 110.49))
-    (stroke (width 0) (type default) (color 0 0 0 0))
-  )
   (wire (pts (xy 135.89 92.71) (xy 139.7 92.71))
     (stroke (width 0) (type default) (color 0 0 0 0))
   )
+  (wire (pts (xy 123.19 90.17) (xy 125.73 90.17))
+    (stroke (width 0) (type default) (color 0 0 0 0))
+  )
   (wire (pts (xy 139.7 90.17) (xy 125.73 90.17))
     (stroke (width 0) (type default) (color 0 0 0 0))
@@
     (stroke (width 0) (type default) (color 0 0 0 0))
   )
-  (wire (pts (xy 116.205 110.49) (xy 116.205 101.6))
+  (wire (pts (xy 104.775 110.49) (xy 104.775 101.6))
+    (stroke (width 0) (type default) (color 0 0 0 0))
+  )
+  (wire (pts (xy 113.03 110.49) (xy 125.73 110.49))
     (stroke (width 0) (type default) (color 0 0 0 0))
   )
@@
     (stroke (width 0) (type default) (color 0 0 0 0))
   )
-  (wire (pts (xy 116.205 90.17) (xy 125.73 90.17))
-    (stroke (width 0) (type default) (color 0 0 0 0))
-  )
   (wire (pts (xy 125.73 90.17) (xy 125.73 99.06))
     (stroke (width 0) (type default) (color 0 0 0 0))
@@
     (stroke (width 0) (type default) (color 0 0 0 0))
   )
+  (wire (pts (xy 115.57 95.25) (xy 113.03 95.25))
+    (stroke (width 0) (type default) (color 0 0 0 0))
+  )
   (wire (pts (xy 153.035 110.49) (xy 139.7 110.49))
     (stroke (width 0) (type default) (color 0 0 0 0))
   )
-  (wire (pts (xy 116.205 99.06) (xy 116.205 90.17))
+  (wire (pts (xy 104.775 99.06) (xy 104.775 90.17))
+    (stroke (width 0) (type default) (color 0 0 0 0))
+  )
+  (wire (pts (xy 104.775 90.17) (xy 115.57 90.17))
+    (stroke (width 0) (type default) (color 0 0 0 0))
+  )
+  (wire (pts (xy 123.19 92.71) (xy 123.19 90.17))
     (stroke (width 0) (type default) (color 0 0 0 0))
   )
@@
     (effects (font (size 1.27 1.27)) (justify left bottom))
   )
-  (text "Output" (at 108.585 105.41 0)
+  (text "Output" (at 95.885 105.41 0)
     (effects (font (size 1.27 1.27)) (justify left bottom))
   )
@@
   )
   (symbol (lib_id "Connector:Screw_Terminal_01x02") (at 168.275 99.06 0) (unit 1)
-    (in_bom yes) (on_board yes) (fields_autoplaced)
-    (property "Reference" "J2" (id 0) (at 170.815 99.0599 0)
+    (in_bom yes) (on_board yes)
+    (property "Reference" "J2" (id 0) (at 167.005 94.615 0)
       (effects (font (size 1.27 1.27)) (justify left))
     )
     (property "Value" "Screw_Terminal_01x02" (id 1) (at 170.815 101.5999 0)
-      (effects (font (size 1.27 1.27)) (justify left))
+      (effects (font (size 1.27 1.27)) (justify left) hide)
     )
     (property "Footprint" "TerminalBlock:TerminalBlock_bornier-2_P5.08mm" (id 2) (at 168.275 99.06 0)
@@
     (pin "2")
   )
+  (symbol (lib_id "SparkFun-Switches:SWITCH-SPDT-PTH-11.6X4.0MM-KIT") (at 120.65 92.71 180) (unit 1)
+    (in_bom yes) (on_board yes) (fields_autoplaced)
+    (property "Reference" "S1" (id 0) (at 119.2403 87.63 0)
+      (effects (font (size 1.143 1.143)))
+    )
+    (property "Value" "SWITCH-SPDT-PTH-11.6X4.0MM-KIT" (id 1) (at 119.2403 86.995 0)
+      (effects (font (size 1.143 1.143)) hide)
+    )
+    (property "Footprint" "SnapEDA Library:SW_1825159-1" (id 2) (at 120.65 99.06 0)
+      (effects (font (size 0.508 0.508)) hide)
+    )
+    (property "Datasheet" "" (id 3) (at 120.65 92.71 0)
+      (effects (font (size 1.27 1.27)) hide)
+    )
+    (property "Field4" "SWCH-08261" (id 4) (at 119.2403 88.265 0)
+      (effects (font (size 1.524 1.524)) hide)
+    )
+    (pin "1")
+    (pin "2")
+    (pin "3")
+  )
   (symbol (lib_id "Device:R") (at 153.035 95.25 0) (unit 1)
     (in_bom yes) (on_board yes) (fields_autoplaced)
@@
     (pin "1")
   )
-  (symbol (lib_id "Connector:Screw_Terminal_01x02") (at 111.125 101.6 180) (unit 1)
-    (in_bom yes) (on_board yes) (fields_autoplaced)
-    (property "Reference" "J1" (id 0) (at 111.125 92.075 0))
-    (property "Value" "Screw_Terminal_01x02" (id 1) (at 111.125 94.615 0))
-    (property "Footprint" "TerminalBlock:TerminalBlock_bornier-2_P5.08mm" (id 2) (at 111.125 101.6 0)
-      (effects (font (size 1.27 1.27)) hide)
-    )
-    (property "Datasheet" "~" (id 3) (at 111.125 101.6 0)
+  (symbol (lib_id "Connector:Screw_Terminal_01x02") (at 99.695 101.6 180) (unit 1)
+    (in_bom yes) (on_board yes) (fields_autoplaced)
+    (property "Reference" "J1" (id 0) (at 99.695 95.25 0))
+    (property "Value" "Screw_Terminal_01x02" (id 1) (at 99.695 94.615 0)
+      (effects (font (size 1.27 1.27)) hide)
+    )
+    (property "Footprint" "TerminalBlock:TerminalBlock_bornier-2_P5.08mm" (id 2) (at 99.695 101.6 0)
+      (effects (font (size 1.27 1.27)) hide)
+    )
+    (property "Datasheet" "~" (id 3) (at 99.695 101.6 0)
       (effects (font (size 1.27 1.27)) hide)
     )
@@
     )
     (property "Datasheet" "~" (id 3) (at 144.145 96.52 0)
+      (effects (font (size 1.27 1.27)) hide)
+    )
+    (pin "1")
+    (pin "2")
+  )
+  (symbol (lib_id "Device:LED") (at 113.03 99.06 90) (unit 1)
+    (in_bom yes) (on_board yes)
+    (property "Reference" "D1" (id 0) (at 107.315 97.79 90)
+      (effects (font (size 1.27 1.27)) (justify right))
+    )
+    (property "Value" "LED" (id 1) (at 107.315 100.33 90)
+      (effects (font (size 1.27 1.27)) (justify right))
+    )
+    (property "Footprint" "LED_THT:LED_D5.0mm_Clear" (id 2) (at 113.03 99.06 0)
+      (effects (font (size 1.27 1.27)) hide)
+    )
+    (property "Datasheet" "~" (id 3) (at 113.03 99.06 0)
+      (effects (font (size 1.27 1.27)) hide)
+    )
+    (pin "1")
+    (pin "2")
+  )
+  (symbol (lib_id "Device:R") (at 113.03 106.68 0) (unit 1)
+    (in_bom yes) (on_board yes)
+    (property "Reference" "R3" (id 0) (at 107.315 105.41 0)
+      (effects (font (size 1.27 1.27)) (justify left))
+    )
+    (property "Value" "300" (id 1) (at 107.315 107.95 0)
+      (effects (font (size 1.27 1.27)) (justify left))
+    )
+    (property "Footprint" "Resistor_THT:R_Axial_DIN0204_L3.6mm_D1.6mm_P7.62mm_Horizontal" (id 2) (at 111.252 106.68 90)
+      (effects (font (size 1.27 1.27)) hide)
+    )
+    (property "Datasheet" "~" (id 3) (at 113.03 106.68 0)
       (effects (font (size 1.27 1.27)) hide)
     )
@@
       (reference "C1") (unit 1) (value "220pf") (footprint "Capacitor_THT:C_Axial_L5.1mm_D3.1mm_P7.50mm_Horizontal")
     )
+    (path "/e027e40e-245b-4b6b-928b-0501a7da5de5"
+      (reference "D1") (unit 1) (value "LED") (footprint "LED_THT:LED_D5.0mm_Clear")
+    )
     (path "/c5208d8c-5be5-4514-b93e-909a9ac14ee6"
       (reference "J1") (unit 1) (value "Screw_Terminal_01x02") (footprint "TerminalBlock:TerminalBlock_bornier-2_P5.08mm")
@@
       (reference "R2") (unit 1) (value "330") (footprint "Resistor_THT:R_Axial_DIN0204_L3.6mm_D1.6mm_P7.62mm_Horizontal")
     )
-  )
+    (path "/fec27d13-0747-41e3-a4d8-e21a45052ada"
+      (reference "R3") (unit 1) (value "300") (footprint "Resistor_THT:R_Axial_DIN0204_L3.6mm_D1.6mm_P7.62mm_Horizontal")
+    )
+    (path "/5a60103d-c1f5-44fb-9ca6-bd09329bef56"
+      (reference "S1") (unit 1) (value "SWITCH-SPDT-PTH-11.6X4.0MM-KIT") (footprint "SnapEDA Library:SW_1825159-1")
+    )
+  )

Commit message: added fabrication files and cleanup
Other:
- title: (none) -> Simple JouleThief 
- moved on the sheet: C1, D1, J1, J2, L1, Q1, Q2, R1, R2, R3, S1

Commit message: smd parts found and added.
Parts:
- C1: footprint Capacitor_THT:C_Axial_L5.1mm_D3.1mm_P7.50mm_Horizontal -> Capacitor_SMD:C_0805_2012Metric_Pad1.18x1.45mm_HandSolder
- D1: footprint LED_THT:LED_D5.0mm_Clear -> LED_SMD:LED_0805_2012Metric_Pad1.15x1.40mm_HandSolder
- L1: footprint Inductor_THT:L_Axial_L5.0mm_D3.6mm_P10.00mm_Horizontal_Murata_BL01RN1A2A2 -> Inductor_SMD:L_6.3x6.3_H3
- Q1, Q2: footprint Package_TO_SOT_THT:TO-92_Inline -> SamacSys_Parts:BC847215
- R1, R2, R3: footprint Resistor_THT:R_Axial_DIN0204_L3.6mm_D1.6mm_P7.62mm_Horizontal -> Resistor_SMD:R_0805_2012Metric_Pad1.20x1.40mm_HandSolder
- S1: footprint SnapEDA Library:SW_1825159-1 -> SamacSys_Parts:LSSM12PVTR
Changed lines of the file:
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@@
       (effects (font (size 1.27 1.27)) (justify left))
     )
-    (property "Footprint" "Package_TO_SOT_THT:TO-92_Inline" (id 2) (at 167.64 107.95 0)
+    (property "Footprint" "SamacSys_Parts:BC847215" (id 2) (at 167.64 107.95 0)
       (effects (font (size 1.27 1.27) italic) (justify left) hide)
     )
@@
     (property "Reference" "L1" (id 0) (at 158.115 84.455 90))
     (property "Value" "100uH" (id 1) (at 158.115 86.995 90))
-    (property "Footprint" "Inductor_THT:L_Axial_L5.0mm_D3.6mm_P10.00mm_Horizontal_Murata_BL01RN1A2A2" (id 2) (at 158.115 90.805 0)
+    (property "Footprint" "Inductor_SMD:L_6.3x6.3_H3" (id 2) (at 158.115 90.805 0)
       (effects (font (size 1.27 1.27)) hide)
     )
@@
       (effects (font (size 1.27 1.27)) (justify left))
     )
-    (property "Footprint" "Package_TO_SOT_THT:TO-92_Inline" (id 2) (at 135.255 106.68 0)
+    (property "Footprint" "SamacSys_Parts:BC847215" (id 2) (at 135.255 106.68 0)
       (effects (font (size 1.27 1.27) italic) (justify left) hide)
     )
@@
       (effects (font (size 1.27 1.27)) (justify left))
     )
-    (property "Footprint" "Capacitor_THT:C_Axial_L5.1mm_D3.1mm_P7.50mm_Horizontal" (id 2) (at 148.9202 100.965 0)
+    (property "Footprint" "Capacitor_SMD:C_0805_2012Metric_Pad1.18x1.45mm_HandSolder" (id 2) (at 148.9202 100.965 0)
       (effects (font (size 1.27 1.27)) hide)
     )
@@
       (effects (font (size 1.143 1.143)) hide)
     )
-    (property "Footprint" "SnapEDA Library:SW_1825159-1" (id 2) (at 132.715 99.695 0)
+    (property "Footprint" "SamacSys_Parts:LSSM12PVTR" (id 2) (at 132.715 99.695 0)
       (effects (font (size 0.508 0.508)) hide)
     )
@@
       (effects (font (size 1.27 1.27)) (justify left))
     )
-    (property "Footprint" "Resistor_THT:R_Axial_DIN0204_L3.6mm_D1.6mm_P7.62mm_Horizontal" (id 2) (at 163.322 95.885 90)
+    (property "Footprint" "Resistor_SMD:R_0805_2012Metric_Pad1.20x1.40mm_HandSolder" (id 2) (at 163.322 95.885 90)
       (effects (font (size 1.27 1.27)) hide)
     )
@@
       (effects (font (size 1.27 1.27)) (justify left))
     )
-    (property "Footprint" "Resistor_THT:R_Axial_DIN0204_L3.6mm_D1.6mm_P7.62mm_Horizontal" (id 2) (at 154.432 97.155 90)
+    (property "Footprint" "Resistor_SMD:R_0805_2012Metric_Pad1.20x1.40mm_HandSolder" (id 2) (at 154.432 97.155 90)
       (effects (font (size 1.27 1.27)) hide)
     )
@@
       (effects (font (size 1.27 1.27)) (justify right))
     )
-    (property "Footprint" "LED_THT:LED_D5.0mm_Clear" (id 2) (at 125.095 99.695 0)
+    (property "Footprint" "LED_SMD:LED_0805_2012Metric_Pad1.15x1.40mm_HandSolder" (id 2) (at 125.095 99.695 0)
       (effects (font (size 1.27 1.27)) hide)
     )
@@
       (effects (font (size 1.27 1.27)) (justify left))
     )
-    (property "Footprint" "Resistor_THT:R_Axial_DIN0204_L3.6mm_D1.6mm_P7.62mm_Horizontal" (id 2) (at 123.317 107.315 90)
+    (property "Footprint" "Resistor_SMD:R_0805_2012Metric_Pad1.20x1.40mm_HandSolder" (id 2) (at 123.317 107.315 90)
       (effects (font (size 1.27 1.27)) hide)
     )
@@
     )
     (path "/56f57a0c-d952-4b14-b499-4833f5f6a321"
-      (reference "C1") (unit 1) (value "220pf") (footprint "Capacitor_THT:C_Axial_L5.1mm_D3.1mm_P7.50mm_Horizontal")
+      (reference "C1") (unit 1) (value "220pf") (footprint "Capacitor_SMD:C_0805_2012Metric_Pad1.18x1.45mm_HandSolder")
     )
     (path "/e027e40e-245b-4b6b-928b-0501a7da5de5"
-      (reference "D1") (unit 1) (value "LED") (footprint "LED_THT:LED_D5.0mm_Clear")
+      (reference "D1") (unit 1) (value "LED") (footprint "LED_SMD:LED_0805_2012Metric_Pad1.15x1.40mm_HandSolder")
     )
     (path "/c5208d8c-5be5-4514-b93e-909a9ac14ee6"
@@
     )
     (path "/41c982a7-98bb-4b69-93c8-cae707855073"
-      (reference "L1") (unit 1) (value "100uH") (footprint "Inductor_THT:L_Axial_L5.0mm_D3.6mm_P10.00mm_Horizontal_Murata_BL01RN1A2A2")
+      (reference "L1") (unit 1) (value "100uH") (footprint "Inductor_SMD:L_6.3x6.3_H3")
     )
     (path "/473a4415-2386-4149-a3fe-7889d826e6e0"
-      (reference "Q1") (unit 1) (value "BC547") (footprint "Package_TO_SOT_THT:TO-92_Inline")
+      (reference "Q1") (unit 1) (value "BC547") (footprint "SamacSys_Parts:BC847215")
     )
     (path "/11a20350-8cce-4cf4-9ca6-d18c48d985d0"
-      (reference "Q2") (unit 1) (value "BC547") (footprint "Package_TO_SOT_THT:TO-92_Inline")
+      (reference "Q2") (unit 1) (value "BC547") (footprint "SamacSys_Parts:BC847215")
     )
     (path "/dfb132cf-0fb7-4414-94e9-dfa0285c3691"
-      (reference "R1") (unit 1) (value "22k") (footprint "Resistor_THT:R_Axial_DIN0204_L3.6mm_D1.6mm_P7.62mm_Horizontal")
+      (reference "R1") (unit 1) (value "22k") (footprint "Resistor_SMD:R_0805_2012Metric_Pad1.20x1.40mm_HandSolder")
     )
     (path "/6469d014-f8d3-4035-9db8-9f9bf2959430"
-      (reference "R2") (unit 1) (value "330") (footprint "Resistor_THT:R_Axial_DIN0204_L3.6mm_D1.6mm_P7.62mm_Horizontal")
+      (reference "R2") (unit 1) (value "330") (footprint "Resistor_SMD:R_0805_2012Metric_Pad1.20x1.40mm_HandSolder")
     )
     (path "/fec27d13-0747-41e3-a4d8-e21a45052ada"
-      (reference "R3") (unit 1) (value "300") (footprint "Resistor_THT:R_Axial_DIN0204_L3.6mm_D1.6mm_P7.62mm_Horizontal")
+      (reference "R3") (unit 1) (value "300") (footprint "Resistor_SMD:R_0805_2012Metric_Pad1.20x1.40mm_HandSolder")
     )
     (path "/5a60103d-c1f5-44fb-9ca6-bd09329bef56"
-      (reference "S1") (unit 1) (value "SWITCH-SPDT-PTH-11.6X4.0MM-KIT") (footprint "SnapEDA Library:SW_1825159-1")
-    )
-  )
+      (reference "S1") (unit 1) (value "SWITCH-SPDT-PTH-11.6X4.0MM-KIT") (footprint "SamacSys_Parts:LSSM12PVTR")
+    )
+  )
